File: LaserDriver.kicad_sch (KiCad schematic)
At the start: 30 parts, among them J100 Screw_Terminal_01x04, J101 Screw_Terminal_01x02, J102 nano_left, J103 nano_right, U100 TPS92513DGQR

Commit message: increased screw size, fixed dimensions
Parts:
- H1, H2, H3: footprint MountingHole:MountingHole_3.2mm_M3 -> MountingHole:MountingHole_4.3mm_M4
Other:
- note added: "M4 Mounting Holes"
- note removed: "M3 Mounting Holes"
Changed lines of the file:
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@@
 		)
 	)
-	(text "M3 Mounting Holes"
+	(text "M4 Mounting Holes"
 		(exclude_from_sim no)
 		(at 167.894 141.224 0)
@@
 		)
 		(instances
-			(project ""
+			(project "LaserDriver"
 				(path "/e8909e30-da70-4cda-aa2c-d92cdd96f174"
 					(reference "J102")
@@
 		)
 		(instances
-			(project ""
+			(project "LaserDriver"
 				(path "/e8909e30-da70-4cda-aa2c-d92cdd96f174"
 					(reference "R107")
@@
 		)
 		(instances
-			(project ""
+			(project "LaserDriver"
 				(path "/e8909e30-da70-4cda-aa2c-d92cdd96f174"
 					(reference "#PWR03")
@@
 		)
 		(instances
-			(project ""
+			(project "LaserDriver"
 				(path "/e8909e30-da70-4cda-aa2c-d92cdd96f174"
 					(reference "#PWR08")
@@
 		)
 		(instances
-			(project ""
+			(project "LaserDriver"
 				(path "/e8909e30-da70-4cda-aa2c-d92cdd96f174"
 					(reference "R109")
@@
 		)
 		(instances
-			(project ""
+			(project "LaserDriver"
 				(path "/e8909e30-da70-4cda-aa2c-d92cdd96f174"
 					(reference "#PWR011")
@@
 		)
 		(instances
-			(project ""
+			(project "LaserDriver"
 				(path "/e8909e30-da70-4cda-aa2c-d92cdd96f174"
 					(reference "#PWR05")
@@
 		)
 		(instances
-			(project ""
+			(project "LaserDriver"
 				(path "/e8909e30-da70-4cda-aa2c-d92cdd96f174"
 					(reference "C104")
@@
 		)
 		(instances
-			(project ""
+			(project "LaserDriver"
 				(path "/e8909e30-da70-4cda-aa2c-d92cdd96f174"
 					(reference "D101")
@@
 		)
 		(instances
-			(project ""
+			(project "LaserDriver"
 				(path "/e8909e30-da70-4cda-aa2c-d92cdd96f174"
 					(reference "#PWR012")
@@
 		)
 		(instances
-			(project ""
+			(project "LaserDriver"
 				(path "/e8909e30-da70-4cda-aa2c-d92cdd96f174"
 					(reference "#PWR06")
@@
 		)
 		(instances
-			(project ""
+			(project "LaserDriver"
 				(path "/e8909e30-da70-4cda-aa2c-d92cdd96f174"
 					(reference "R104")
@@
 		)
 		(instances
-			(project ""
+			(project "LaserDriver"
 				(path "/e8909e30-da70-4cda-aa2c-d92cdd96f174"
 					(reference "R105")
@@
 		)
 		(instances
-			(project ""
+			(project "LaserDriver"
 				(path "/e8909e30-da70-4cda-aa2c-d92cdd96f174"
 					(reference "J101")
@@
 		)
 		(instances
-			(project ""
+			(project "LaserDriver"
 				(path "/e8909e30-da70-4cda-aa2c-d92cdd96f174"
 					(reference "C102")
@@
 		)
 		(instances
-			(project ""
+			(project "LaserDriver"
 				(path "/e8909e30-da70-4cda-aa2c-d92cdd96f174"
 					(reference "D102")
@@
 		)
 		(instances
-			(project ""
+			(project "LaserDriver"
 				(path "/e8909e30-da70-4cda-aa2c-d92cdd96f174"
 					(reference "#PWR013")
@@
 		)
 		(instances
-			(project ""
+			(project "LaserDriver"
 				(path "/e8909e30-da70-4cda-aa2c-d92cdd96f174"
 					(reference "#FLG01")
@@
 		)
 		(instances
-			(project ""
+			(project "LaserDriver"
 				(path "/e8909e30-da70-4cda-aa2c-d92cdd96f174"
 					(reference "#FLG04")
@@
 		)
 		(instances
-			(project ""
+			(project "LaserDriver"
 				(path "/e8909e30-da70-4cda-aa2c-d92cdd96f174"
 					(reference "#FLG02")
@@
 		)
 		(instances
-			(project ""
+			(project "LaserDriver"
 				(path "/e8909e30-da70-4cda-aa2c-d92cdd96f174"
 					(reference "R108")
@@
 		)
 		(instances
-			(project ""
+			(project "LaserDriver"
 				(path "/e8909e30-da70-4cda-aa2c-d92cdd96f174"
 					(reference "D100")
@@
 			)
 		)
-		(property "Footprint" "MountingHole:MountingHole_3.2mm_M3"
+		(property "Footprint" "MountingHole:MountingHole_4.3mm_M4"
 			(at 161.29 149.86 0)
 			(effects
@@
 		)
 		(instances
-			(project ""
+			(project "LaserDriver"
 				(path "/e8909e30-da70-4cda-aa2c-d92cdd96f174"
 					(reference "R111")
@@
 		)
 		(instances
-			(project ""
+			(project "LaserDriver"
 				(path "/e8909e30-da70-4cda-aa2c-d92cdd96f174"
 					(reference "C105")
@@
 		)
 		(instances
-			(project ""
+			(project "LaserDriver"
 				(path "/e8909e30-da70-4cda-aa2c-d92cdd96f174"
 					(reference "R112")
@@
 		)
 		(instances
-			(project ""
+			(project "LaserDriver"
 				(path "/e8909e30-da70-4cda-aa2c-d92cdd96f174"
 					(reference "R106")
@@
 		)
 		(instances
-			(project ""
+			(project "LaserDriver"
 				(path "/e8909e30-da70-4cda-aa2c-d92cdd96f174"
 					(reference "R110")
@@
 		)
 		(instances
-			(project ""
+			(project "LaserDriver"
 				(path "/e8909e30-da70-4cda-aa2c-d92cdd96f174"
 					(reference "C103")
@@
 		)
 		(instances
-			(project ""
+			(project "LaserDriver"
 				(path "/e8909e30-da70-4cda-aa2c-d92cdd96f174"
 					(reference "L100")
@@
 		)
 		(instances
-			(project ""
+			(project "LaserDriver"
 				(path "/e8909e30-da70-4cda-aa2c-d92cdd96f174"
 					(reference "#PWR09")
@@
 		)
 		(instances
-			(project ""
+			(project "LaserDriver"
 				(path "/e8909e30-da70-4cda-aa2c-d92cdd96f174"
 					(reference "#PWR04")
@@
 			)
 		)
-		(property "Footprint" "MountingHole:MountingHole_3.2mm_M3"
+		(property "Footprint" "MountingHole:MountingHole_4.3mm_M4"
 			(at 161.29 144.78 0)
 			(effects
@@
 		)
 		(instances
-			(project ""
+			(project "LaserDriver"
 				(path "/e8909e30-da70-4cda-aa2c-d92cdd96f174"
 					(reference "H1")
@@
 		)
 		(instances
-			(project ""
+			(project "LaserDriver"
 				(path "/e8909e30-da70-4cda-aa2c-d92cdd96f174"
 					(reference "#PWR01")
@@
 		)
 		(instances
-			(project ""
+			(project "LaserDriver"
 				(path "/e8909e30-da70-4cda-aa2c-d92cdd96f174"
 					(reference "J100")
@@
 		)
 		(instances
-			(project ""
+			(project "LaserDriver"
 				(path "/e8909e30-da70-4cda-aa2c-d92cdd96f174"
 					(reference "R103")
@@
 		)
 		(instances
-			(project ""
+			(project "LaserDriver"
 				(path "/e8909e30-da70-4cda-aa2c-d92cdd96f174"
 					(reference "U100")
@@
 		)
 		(instances
-			(project ""
+			(project "LaserDriver"
 				(path "/e8909e30-da70-4cda-aa2c-d92cdd96f174"
 					(reference "C100")
@@
 		)
 		(instances
-			(project ""
+			(project "LaserDriver"
 				(path "/e8909e30-da70-4cda-aa2c-d92cdd96f174"
 					(reference "#PWR010")
@@
 			)
 		)
-		(property "Footprint" "MountingHole:MountingHole_3.2mm_M3"
+		(property "Footprint" "MountingHole:MountingHole_4.3mm_M4"
 			(at 161.29 154.94 0)
 			(effects
@@
 		)
 		(instances
-			(project ""
+			(project "LaserDriver"
 				(path "/e8909e30-da70-4cda-aa2c-d92cdd96f174"
 					(reference "#PWR02")
@@
 		)
 		(instances
-			(project ""
+			(project "LaserDriver"
 				(path "/e8909e30-da70-4cda-aa2c-d92cdd96f174"
 					(reference "#FLG03")
@@
 		)
 		(instances
-			(project ""
+			(project "LaserDriver"
 				(path "/e8909e30-da70-4cda-aa2c-d92cdd96f174"
 					(reference "C106")
