File: LaserDriver.kicad_sch (KiCad schematic)
At the start: 30 parts, among them J100 Screw_Terminal_01x04, J101 Screw_Terminal_01x02, J102 nano_left, J103 nano_right, U100 TPS92513DGQR

Commit message: Fixed supplier and manufacturer issues
Parts:
- L100: footprint Inductor_SMD:L_7.3x7.3_H4.5 -> Inductor_SMD:L_Bourns_SRP7028A_7.3x6.6mm; Manufacturer PULSE -> BOURNS; Manufacturer Part Number PA4308.333NLT -> SRP7028A-330M
Changed lines of the file:
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@@
 			)
 		)
-		(property "Footprint" "Inductor_SMD:L_7.3x7.3_H4.5"
+		(property "Footprint" "Inductor_SMD:L_Bourns_SRP7028A_7.3x6.6mm"
 			(at 139.7 39.37 0)
 			(effects
@@
 			)
 		)
-		(property "Manufacturer" "PULSE"
+		(property "Manufacturer" "BOURNS"
 			(at 139.7 39.37 90)
 			(effects
@@
 			)
 		)
-		(property "Manufacturer Part Number" "PA4308.333NLT"
+		(property "Manufacturer Part Number" "SRP7028A-330M"
 			(at 139.7 39.37 90)
 			(effects
