File: LaserDriver.kicad_pcb (KiCad board)
At the start: 2 copper layers, 39.5 x 40 mm, 30 parts, among them J100 Screw_Terminal_01x04, J101 Screw_Terminal_01x02, J102 nano_left, J103 nano_right, U100 TPS92513DGQR

Commit message: fixed errors
Parts:
- U100: footprint TPS:DGQ0010D_L -> TPS:DGQ0010D_NV_L
- moved J101 2.57 mm to (65.5, 115.5), turned to 90 degrees
- moved D100 0.61 mm to (31.8, 106.3), turned to -90 degrees
Connections:
- C104 pad 2: Net-(J101-Pin_2) -> Net-(J101-Pin_1)
- J101 pad 1: Net-(D102-K) -> Net-(J101-Pin_1)
- J101 pad 2: Net-(J101-Pin_2) -> Net-(D102-K)
- R104 pad 2: Net-(J101-Pin_2) -> Net-(J101-Pin_1)
- R105 pad 1: Net-(J101-Pin_2) -> Net-(J101-Pin_1)
Routing:
- net Net-(J101-Pin_1): track 0.00 -> 18.2 mm
- net Net-(J101-Pin_2): track 18.2 -> 0.00 mm
- net GND: track 34.7 -> 39.1 mm, vias 15 -> 18
- net Net-(J100-Pin_2): track 0.00 -> 2.54 mm
Other:
- board size 39.5 x 40 mm -> 40.2 x 40.5 mm
